File: AC_power_module.kicad_sch (KiCad schematic)
At the start: 8 parts, among them J301 7.62mm 2-Pin Screw Terminal

Commit message: "Assign Footprints Done"
Parts:
- removed RV301: 10D561, Varistor:RV_Disc_D12mm_W5.1mm_P7.5mm, symbol Device:Varistor
- added RV401: Varistor, Varistor:RV_Disc_D12mm_W5.1mm_P7.5mm, symbol Device:Varistor
- C402: footprint Capacitor_SMD:C_0402_1005Metric_Pad0.74x0.62mm_HandSolder -> Capacitor_SMD:C_0603_1608Metric_Pad1.08x0.95mm_HandSolder
- C403: footprint Capacitor_SMD:C_0805_2012Metric_Pad1.18x1.45mm_HandSolder -> Capacitor_SMD:C_0603_1608Metric_Pad1.08x0.95mm_HandSolder
- FL401: renamed from FL301; footprint SamacSys_Parts:B82730U3951A020 -> govi_v3_SHT41_sensor_kicad:B82730U3451A020-ferrite-core-inductor
- J401: renamed from J301; footprint govi.ai-sensor-sht41-wifi:P=7.62mm Barrier Terminal Blocks -> govi_v3_SHT41_sensor_kicad:P=7.62mm Barrier Terminal Blocks azend
- TH401: renamed from TH301; footprint SamacSys_Parts:B57236S0250M000 -> govi_v3_SHT41_sensor_kicad:B57236S0250M000-Thermister
Connections:
- net at C401.1, FL401.2, TH401.2: now also RV401.1
- net at C401.2, FL401.1, J401.1 (Pin_1): now also RV401.2
Changed lines of the file:
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@@
+	)
+	(symbol
+		(lib_name "Varistor_1")
+		(lib_id "Device:Varistor")
+		(at 85.09 97.79 0)
+		(unit 1)
+		(exclude_from_sim no)
+		(in_bom yes)
+		(on_board yes)
+		(dnp no)
+		(fields_autoplaced yes)
+		(property "Reference" "RV401"
+			(at 87.63 96.7132 0)
+			(effects
+				(font
+					(size 1.27 1.27)
+				)
+				(justify left)
+			)
+		)
+		(property "Value" "Varistor"
+			(at 87.63 99.2532 0)
+			(effects
+				(font
+					(size 1.27 1.27)
+				)
+				(justify left)
+			)
+		)
+		(property "Footprint" "Varistor:RV_Disc_D12mm_W5.1mm_P7.5mm"
+			(at 83.312 97.79 90)
+			(effects
+				(font
+					(size 1.27 1.27)
+				)
+				(hide yes)
+			)
+		)
+		(property "Datasheet" "~"
+			(at 85.09 97.79 0)
+			(effects
+				(font
+					(size 1.27 1.27)
+				)
+				(hide yes)
+			)
+		)
+		(property "Description" "Voltage dependent resistor"
+			(at 85.09 97.79 0)
+			(effects
+				(font
+					(size 1.27 1.27)
+				)
+				(hide yes)
+			)
+		)
+		(property "Sim.Name" "kicad_builtin_varistor"
+			(at 85.09 97.79 0)
+			(effects
+				(font
+					(size 1.27 1.27)
+				)
+				(hide yes)
+			)
+		)
+		(property "Sim.Device" "SUBCKT"
+			(at 85.09 97.79 0)
+			(effects
+				(font
+					(size 1.27 1.27)
+				)
+				(hide yes)
+			)
+		)
+		(property "Sim.Pins" "1=A 2=B"
+			(at 85.09 97.79 0)
+			(effects
+				(font
+					(size 1.27 1.27)
+				)
+				(hide yes)
+			)
+		)
+		(property "Sim.Params" "threshold=1k"
+			(at 85.09 97.79 0)
+			(effects
+				(font
+					(size 1.27 1.27)
+				)
+				(hide yes)
+			)
+		)
+		(property "Sim.Library" "${KICAD9_SYMBOL_DIR}/Simulation_SPICE.sp"
+			(at 85.09 97.79 0)
+			(effects
+				(font
+					(size 1.27 1.27)
+				)
+				(hide yes)
+			)
+		)
+		(pin "1"
+		)
+		(pin "2"
+		)
+		(instances
+			(project ""
+				(path "/ba95ddf4-72c6-4eeb-9c09-ae7c8e5af670/5ca2b3fd-61f6-48b4-88ce-6504da0079e1"
+					(reference "RV401")
+					(unit 1)
+				)
+			)
+		)
 	)
 	(symbol
@@
 		(dnp no)
 		(fields_autoplaced yes)
-		(property "Reference" "#FLG0402"
+		(property "Reference" "#FLG0401"
 			(at 152.4 86.995 0)
 			(effects
@@
 			(project "govi_v3_SHT41_sensor_kicad"
 				(path "/ba95ddf4-72c6-4eeb-9c09-ae7c8e5af670/5ca2b3fd-61f6-48b4-88ce-6504da0079e1"
-					(reference "#FLG0402")
+					(reference "#FLG0401")
 					(unit 1)
 				)
@@
 		(on_board yes)
 		(dnp no)
-		(property "Reference" "FL301"
+		(property "Reference" "FL401"
 			(at 138.43 88.9 0)
 			(effects
@@
 			)
 		)
-		(property "Footprint" "SamacSys_Parts:B82730U3951A020"
+		(property "Footprint" "govi_v3_SHT41_sensor_kicad:B82730U3451A020-ferrite-core-inductor"
 			(at 137.16 104.14 0)
 			(effects
@@
 			(project "govi_v3_SHT41_sensor_kicad"
 				(path "/ba95ddf4-72c6-4eeb-9c09-ae7c8e5af670/5ca2b3fd-61f6-48b4-88ce-6504da0079e1"
-					(reference "FL301")
+					(reference "FL401")
 					(unit 1)
 				)
@@
 			)
 		)
-		(property "Footprint" "Capacitor_SMD:C_0402_1005Metric_Pad0.74x0.62mm_HandSolder"
+		(property "Footprint" "Capacitor_SMD:C_0603_1608Metric_Pad1.08x0.95mm_HandSolder"
 			(at 213.0552 100.33 0)
 			(effects
@@
 		(dnp no)
 		(fields_autoplaced yes)
-		(property "Reference" "#PWR0405"
+		(property "Reference" "#PWR0406"
 			(at 240.03 113.03 0)
 			(effects
@@
 			(project "govi_v3_SHT41_sensor_kicad"
 				(path "/ba95ddf4-72c6-4eeb-9c09-ae7c8e5af670/5ca2b3fd-61f6-48b4-88ce-6504da0079e1"
-					(reference "#PWR0405")
+					(reference "#PWR0406")
 					(unit 1)
 				)
@@
 		(on_board yes)
 		(dnp no)
-		(property "Reference" "J301"
+		(property "Reference" "J401"
 			(at 60.96 90.17 0)
 			(effects
@@
 			)
 		)
-		(property "Footprint" "govi.ai-sensor-sht41-wifi:P=7.62mm Barrier Terminal Blocks"
+		(property "Footprint" "govi_v3_SHT41_sensor_kicad:P=7.62mm Barrier Terminal Blocks azend"
 			(at 60.96 99.06 0)
 			(effects
@@
 			(project "govi_v3_SHT41_sensor_kicad"
 				(path "/ba95ddf4-72c6-4eeb-9c09-ae7c8e5af670/5ca2b3fd-61f6-48b4-88ce-6504da0079e1"
-					(reference "J301")
+					(reference "J401")
 					(unit 1)
 				)
@@
 		(dnp no)
 		(fields_autoplaced yes)
-		(property "Reference" "#FLG0403"
+		(property "Reference" "#FLG0402"
 			(at 157.48 86.995 0)
 			(effects
@@
 			(project "govi_v3_SHT41_sensor_kicad"
 				(path "/ba95ddf4-72c6-4eeb-9c09-ae7c8e5af670/5ca2b3fd-61f6-48b4-88ce-6504da0079e1"
-					(reference "#FLG0403")
+					(reference "#FLG0402")
 					(unit 1)
 				)
@@
 		(dnp no)
 		(fields_autoplaced yes)
-		(property "Reference" "#PWR0403"
+		(property "Reference" "#PWR0405"
 			(at 240.03 92.71 0)
 			(effects
@@
 			(project "govi_v3_SHT41_sensor_kicad"
 				(path "/ba95ddf4-72c6-4eeb-9c09-ae7c8e5af670/5ca2b3fd-61f6-48b4-88ce-6504da0079e1"
-					(reference "#PWR0403")
+					(reference "#PWR0405")
 					(unit 1)
 				)
@@
 		(dnp no)
 		(fields_autoplaced yes)
-		(property "Reference" "#PWR0407"
+		(property "Reference" "#PWR0403"
 			(at 212.09 92.71 0)
 			(effects
@@
 			(project "govi_v3_SHT41_sensor_kicad"
 				(path "/ba95ddf4-72c6-4eeb-9c09-ae7c8e5af670/5ca2b3fd-61f6-48b4-88ce-6504da0079e1"
-					(reference "#PWR0407")
+					(reference "#PWR0403")
 					(unit 1)
 				)
@@
 			)
 		)
-		(property "Footprint" "Capacitor_SMD:C_0805_2012Metric_Pad1.18x1.45mm_HandSolder"
+		(property "Footprint" "Capacitor_SMD:C_0603_1608Metric_Pad1.08x0.95mm_HandSolder"
 			(at 240.9952 100.33 0)
 			(effects
@@
 	)
 	(symbol
-		(lib_id "Device:Varistor")
-		(at 85.09 97.79 180)
-		(unit 1)
-		(exclude_from_sim no)
-		(in_bom yes)
-		(on_board yes)
-		(dnp no)
-		(fields_autoplaced yes)
-		(property "Reference" "RV301"
-			(at 88.9 96.3267 0)
-			(effects
-				(font
-					(size 1.27 1.27)
-				)
-				(justify right)
-			)
-		)
-		(property "Value" "10D561"
-			(at 88.9 98.8667 0)
-			(effects
-				(font
-					(size 1.27 1.27)
-				)
-				(justify right)
-			)
-		)
-		(property "Footprint" "Varistor:RV_Disc_D12mm_W5.1mm_P7.5mm"
-			(at 86.868 97.79 90)
-			(effects
-				(font
-					(size 1.27 1.27)
-				)
-				(hide yes)
-			)
-		)
-		(property "Datasheet" "~"
-			(at 85.09 97.79 0)
-			(effects
-				(font
-					(size 1.27 1.27)
-				)
-				(hide yes)
-			)
-		)
-		(property "Description" ""
-			(at 85.09 97.79 0)
-			(effects
-				(font
-					(size 1.27 1.27)
-				)
-			)
-		)
-		(property "Sim.Name" "kicad_builtin_varistor"
-			(at 85.09 97.79 0)
-			(effects
-				(font
-					(size 1.27 1.27)
-				)
-				(hide yes)
-			)
-		)
-		(property "Sim.Device" "SUBCKT"
-			(at 85.09 97.79 0)
-			(effects
-				(font
-					(size 1.27 1.27)
-				)
-				(hide yes)
-			)
-		)
-		(property "Sim.Pins" "1=A 2=B"
-			(at 85.09 97.79 0)
-			(effects
-				(font
-					(size 1.27 1.27)
-				)
-				(hide yes)
-			)
-		)
-		(property "Sim.Params" "threshold=1k"
-			(at 85.09 97.79 0)
-			(effects
-				(font
-					(size 1.27 1.27)
-				)
-				(hide yes)
-			)
-		)
-		(property "Sim.Library" "${KICAD7_SYMBOL_DIR}/Simulation_SPICE.sp"
-			(at 85.09 97.79 0)
-			(effects
-				(font
-					(size 1.27 1.27)
-				)
-				(hide yes)
-			)
-		)
-		(pin "1"
-		)
-		(pin "2"
-		)
-		(instances
-			(project "govi_v3_SHT41_sensor_kicad"
-				(path "/ba95ddf4-72c6-4eeb-9c09-ae7c8e5af670/5ca2b3fd-61f6-48b4-88ce-6504da0079e1"
-					(reference "RV301")
-					(unit 1)
-				)
-			)
-		)
-	)
-	(symbol
 		(lib_id "power:+5V")
 		(at 185.42 88.9 0)
@@
 		(dnp no)
 		(fields_autoplaced yes)
-		(property "Reference" "TH301"
+		(property "Reference" "TH401"
 			(at 77.47 83.82 90)
 			(effects
@@
 			)
 		)
-		(property "Footprint" "SamacSys_Parts:B57236S0250M000"
+		(property "Footprint" "govi_v3_SHT41_sensor_kicad:B57236S0250M000-Thermister"
 			(at 77.47 90.17 0)
 			(effects
@@
 			(project "govi_v3_SHT41_sensor_kicad"
 				(path "/ba95ddf4-72c6-4eeb-9c09-ae7c8e5af670/5ca2b3fd-61f6-48b4-88ce-6504da0079e1"
-					(reference "TH301")
-					(unit 1)
-				)
+					(reference "TH401")
+					(unit 1)
+				)

Commit message: "I2c Pin change. PB6:SCL1 , PB7:SDA1"
Parts:
- PS401: footprint Converter_ACDC:Converter_ACDC_Hi-Link_HLK-5Mxx -> govi_v3_SHT41_sensor_kicad:HLK5M05
Changed lines of the file:
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@@
 			)
 		)
-		(property "Footprint" "Converter_ACDC:Converter_ACDC_Hi-Link_HLK-5Mxx"
+		(property "Footprint" "govi_v3_SHT41_sensor_kicad:HLK5M05"
 			(at 168.91 105.41 0)
 			(effects

Commit message: "PCB front Layer Component assembly done"
Parts:
- removed C402: 0.1MFD/16V, Capacitor_SMD:C_0603_1608Metric_Pad1.08x0.95mm_HandSolder, symbol Device:C
- removed C403: 10MFD/16V, Capacitor_SMD:C_0603_1608Metric_Pad1.08x0.95mm_HandSolder, symbol Device:C
- added TP401: 5V, TestPoint:TestPoint_Pad_D1.0mm, symbol Connector:TestPoint
Connections:
- net +5V: now also TP401.1

Commit message: "Routing done. DRC pending"
Other:
- moved on the sheet: C401, FL401, J401, PS401, RV401, TH401, TP401
