File: MPPT_Charger_module.kicad_sch (KiCad schematic)
At the start: 20 parts, among them J501 7.62mm 2-Pin Screw Terminal, J502 Conn_02x02_Odd_Even, Q502 Q_PMOS_Depletion, U501 CN3791

Commit message: "Assign Footprints Done"
Parts:
- C501: renamed from C505; footprint (none) -> Capacitor_SMD:C_0603_1608Metric_Pad1.08x0.95mm_HandSolder
- C502: renamed from C506; footprint (none) -> Capacitor_SMD:C_0603_1608Metric_Pad1.08x0.95mm_HandSolder
- C503: renamed from C501; footprint (none) -> Capacitor_SMD:C_0603_1608Metric_Pad1.08x0.95mm_HandSolder
- C504: renamed from C507; footprint (none) -> Capacitor_SMD:C_0603_1608Metric_Pad1.08x0.95mm_HandSolder
- C505: renamed from C502; footprint (none) -> Capacitor_SMD:C_0603_1608Metric_Pad1.08x0.95mm_HandSolder
- C506: renamed from C503; footprint (none) -> Capacitor_SMD:C_0603_1608Metric_Pad1.08x0.95mm_HandSolder
- C507: renamed from C504; footprint (none) -> Capacitor_SMD:C_0603_1608Metric_Pad1.08x0.95mm_HandSolder
- D501: renamed from D502; footprint (none) -> Diode_SMD:D_SMA
- D502: renamed from D501; footprint (none) -> Diode_SMD:D_SMA
- D503: footprint (none) -> Diode_SMD:D_SMA
- J501: footprint govi.ai-sensor-sht41-wifi:P=7.62mm Barrier Terminal Blocks -> govi_v3_SHT41_sensor_kicad:P=7.62mm Barrier Terminal Blocks azend
- J502: footprint (none) -> Connector_PinHeader_2.54mm:PinHeader_2x04_P2.54mm_Vertical
- L501: footprint (none) -> Inductor_SMD:L_12x12mm_H4.5mm
- Q501: renamed from Q502; footprint (none) -> Package_TO_SOT_SMD:TO-252-2
- R501: renamed from R502; footprint (none) -> Resistor_SMD:R_0603_1608Metric_Pad0.98x0.95mm_HandSolder
- R502: renamed from R501; footprint (none) -> Resistor_SMD:R_0603_1608Metric_Pad0.98x0.95mm_HandSolder
- R503: footprint (none) -> Resistor_SMD:R_0603_1608Metric_Pad0.98x0.95mm_HandSolder
- R504: renamed from R505; footprint (none) -> Resistor_SMD:R_0603_1608Metric_Pad0.98x0.95mm_HandSolder
- R505: renamed from R504; footprint (none) -> Resistor_SMD:R_2512_6332Metric_Pad1.40x3.35mm_HandSolder
Other:
- note added: "- Resistors & Capacitor size - 0603"

Commit message: "Some Component values were changed in MPPT sheet"
Parts:
- C502: value 1uF -> 47nF
- C503: value 220uF 50V -> 220uF 35V; footprint Capacitor_SMD:C_0603_1608Metric_Pad1.08x0.95mm_HandSolder -> Capacitor_SMD:CP_Elec_6.3x7.7
- C507: value 10uF 25V -> 10uF 20V; footprint Capacitor_SMD:C_0603_1608Metric_Pad1.08x0.95mm_HandSolder -> Capacitor_Tantalum_SMD:CP_EIA-3216-18_Kemet-A_HandSolder
- J502: footprint Connector_PinHeader_2.54mm:PinHeader_2x04_P2.54mm_Vertical -> Connector_PinHeader_2.54mm:PinHeader_2x02_P2.54mm_Vertical
Other:
- note added: "- C507 - Tantalum capacitor - T491A106M020AT"
- note removed: "Tantalum capacitor"
Changed lines of the file:
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@@
 		)
 	)
-	(text "Tantalum\ncapacitor"
-		(exclude_from_sim no)
-		(at 245.364 90.678 0)
+	(text "- C507 - Tantalum capacitor - T491A106M020AT"
+		(exclude_from_sim no)
+		(at 41.148 188.722 0)
 		(effects
 			(font
@@
 			)
 		)
-		(property "Value" "10uF 25V"
+		(property "Value" "10uF 20V"
 			(at 241.3 86.9949 0)
 			(effects
@@
 			)
 		)
-		(property "Footprint" "Capacitor_SMD:C_0603_1608Metric_Pad1.08x0.95mm_HandSolder"
+		(property "Footprint" "Capacitor_Tantalum_SMD:CP_EIA-3216-18_Kemet-A_HandSolder"
 			(at 237.49 86.36 0)
 			(effects
@@
 			)
 		)
-		(property "Value" "220uF 50V"
+		(property "Value" "220uF 35V"
 			(at 83.82 86.9949 0)
 			(effects
@@
 			)
 		)
-		(property "Footprint" "Capacitor_SMD:C_0603_1608Metric_Pad1.08x0.95mm_HandSolder"
+		(property "Footprint" "Capacitor_SMD:CP_Elec_6.3x7.7"
 			(at 80.01 86.36 0)
 			(effects
@@
 			)
 		)
-		(property "Value" "1uF"
+		(property "Value" "47nF"
 			(at 73.66 95.2499 0)
 			(effects
@@
 			)
 		)
-		(property "Footprint" "Connector_PinHeader_2.54mm:PinHeader_2x04_P2.54mm_Vertical"
+		(property "Footprint" "Connector_PinHeader_2.54mm:PinHeader_2x02_P2.54mm_Vertical"
 			(at 139.7 88.9 0)
 			(effects

Commit message: "PCB front Layer Component assembly done"
Parts:
- removed J502: Conn_02x02_Odd_Even, Connector_PinHeader_2.54mm:PinHeader_2x02_P2.54mm_Vertical, symbol Connector_Generic:Conn_02x02_Odd_Even
- removed R504: 36K, Resistor_SMD:R_0603_1608Metric_Pad0.98x0.95mm_HandSolder, symbol Device:R
- added TP501: MPPT, TestPoint:TestPoint_Pad_D1.0mm, symbol Connector:TestPoint
- renumbered R505 to R504
Connections:
- net +12V: now also R502.1
- net MPPT+: now also TP501.1
Other:
- note removed: "6V"
- moved on the sheet: R502

Commit message: "Working on Routing MCU"
Parts:
- removed D501: SS54, Diode_SMD:D_SMA, symbol Device:D_Schottky
Connections:
- net +12V: now also Q501.3 (S); no longer Q501.S
- net at D502.1 (K), L501.1: now also Q501.2 (D)
- net at U501.10 (DRV): now also Q501.1 (G); no longer Q501.G
Changed lines of the file:
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@@
 	(wire
 		(pts
-			(xy 160.02 78.74) (xy 162.56 78.74)
+			(xy 160.02 78.74) (xy 173.99 78.74)
 		)
 		(stroke
@@
 		(pts
 			(xy 59.69 90.17) (xy 59.69 100.33)
-		)
-		(stroke
-			(width 0)
-			(type solid)
-		)
-	)
-	(wire
-		(pts
-			(xy 170.18 78.74) (xy 173.99 78.74)
 		)
 		(stroke
@@
 			)
 		)
-		(pin "S"
-		)
-		(pin "D"
-		)
-		(pin "G"
+		(pin "1"
+		)
+		(pin "3"
+		)
+		(pin "2"
 		)
 		(instances
@@
 					(unit 1)
 				)
-			)
-		)
-	)
-	(symbol
-		(lib_id "Device:D_Schottky")
-		(at 166.37 78.74 180)
-		(unit 1)
-		(exclude_from_sim no)
-		(in_bom yes)
-		(on_board yes)
-		(dnp no)
-		(fields_autoplaced yes)
-		(property "Reference" "D501"
-			(at 166.6875 72.39 0)
-			(effects
-				(font
-					(size 1.27 1.27)
-				)
-			)
-		)
-		(property "Value" "SS54"
-			(at 166.6875 74.93 0)
-			(effects
-				(font
-					(size 1.27 1.27)
-				)
-			)
-		)
-		(property "Footprint" "Diode_SMD:D_SMA"
-			(at 166.37 78.74 0)
-			(effects
-				(font
-					(size 1.27 1.27)
-				)
-				(hide yes)
-			)
-		)
-		(property "Datasheet" "~"
-			(at 166.37 78.74 0)
-			(effects
-				(font
-					(size 1.27 1.27)
-				)
-				(hide yes)
-			)
-		)
-		(property "Description" "Schottky diode"
-			(at 166.37 78.74 0)
-			(effects
-				(font
-					(size 1.27 1.27)
-				)
-				(hide yes)
-			)
-		)
-		(pin "2"
-		)
-		(pin "1"
-		)
-		(instances
-			(project "govi_v3_SHT41_sensor_kicad"
-				(path "/ba95ddf4-72c6-4eeb-9c09-ae7c8e5af670/ae21eb8a-dcd5-4896-ab16-4532b352bb44"
-					(reference "D501")
-					(unit 1)
-				)

Commit message: "Before changing the orientation of the LoRa module. removing existing LoRa module routing."
Connections:
- net MPPT+: no longer TP501.1
- net at C506.1, C507.1, D503.2 (A)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: now also TP501.1
Other:
- moved on the sheet: TP501
Changed lines of the file:
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@@
-	)
-	(junction
-		(at 257.81 78.74)
-		(diameter 0)
-		(color 0 0 0 0)
 	)
 	(junction
@@
 	)
 	(junction
+		(at 240.03 78.74)
+		(diameter 0)
+		(color 0 0 0 0)
+	)
+	(junction
 		(at 237.49 96.52)
 		(diameter 0)
@@
 	(wire
 		(pts
+			(xy 240.03 78.74) (xy 247.65 78.74)
+		)
+		(stroke
+			(width 0)
+			(type solid)
+		)
+	)
+	(wire
+		(pts
 			(xy 80.01 100.33) (xy 69.85 100.33)
 		)
@@
 	(wire
 		(pts
+			(xy 240.03 74.93) (xy 240.03 78.74)
+		)
+		(stroke
+			(width 0)
+			(type default)
+		)
+	)
+	(wire
+		(pts
 			(xy 125.73 107.95) (xy 125.73 78.74)
 		)
@@
 	(wire
 		(pts
-			(xy 257.81 78.74) (xy 260.35 78.74)
+			(xy 255.27 78.74) (xy 260.35 78.74)
 		)
 		(stroke
@@
 	(wire
 		(pts
-			(xy 257.81 74.93) (xy 257.81 78.74)
+			(xy 125.73 78.74) (xy 139.7 78.74)
+		)
+		(stroke
+			(width 0)
+			(type solid)
+		)
+	)
+	(wire
+		(pts
+			(xy 222.25 82.55) (xy 222.25 78.74)
+		)
+		(stroke
+			(width 0)
+			(type solid)
+		)
+	)
+	(wire
+		(pts
+			(xy 173.99 78.74) (xy 182.88 78.74)
 		)
 		(stroke
@@
 	(wire
 		(pts
-			(xy 255.27 78.74) (xy 257.81 78.74)
-		)
-		(stroke
-			(width 0)
-			(type solid)
-		)
-	)
-	(wire
-		(pts
-			(xy 125.73 78.74) (xy 139.7 78.74)
-		)
-		(stroke
-			(width 0)
-			(type solid)
-		)
-	)
-	(wire
-		(pts
-			(xy 222.25 82.55) (xy 222.25 78.74)
-		)
-		(stroke
-			(width 0)
-			(type solid)
-		)
-	)
-	(wire
-		(pts
-			(xy 173.99 78.74) (xy 182.88 78.74)
+			(xy 50.8 81.28) (xy 50.8 90.17)
+		)
+		(stroke
+			(width 0)
+			(type solid)
+		)
+	)
+	(polyline
+		(pts
+			(xy 18.415 63.246) (xy 277.114 63.246)
+		)
+		(stroke
+			(width 0)
+			(type dash)
+		)
+	)
+	(wire
+		(pts
+			(xy 80.01 78.74) (xy 80.01 82.55)
 		)
 		(stroke
@@
 	(wire
 		(pts
-			(xy 50.8 81.28) (xy 50.8 90.17)
+			(xy 198.12 110.49) (xy 198.12 78.74)
+		)
+		(stroke
+			(width 0)
+			(type solid)
+		)
+	)
+	(wire
+		(pts
+			(xy 139.7 115.57) (xy 139.7 119.38)
+		)
+		(stroke
+			(width 0)
+			(type solid)
+		)
+	)
+	(wire
+		(pts
+			(xy 222.25 78.74) (xy 217.17 78.74)
+		)
+		(stroke
+			(width 0)
+			(type solid)
+		)
+	)
+	(wire
+		(pts
+			(xy 237.49 96.52) (xy 237.49 90.17)
+		)
+		(stroke
+			(width 0)
+			(type solid)
+		)
+	)
+	(wire
+		(pts
+			(xy 100.33 85.09) (xy 100.33 78.74)
+		)
+		(stroke
+			(width 0)
+			(type solid)
+		)
+	)
+	(wire
+		(pts
+			(xy 173.99 93.98) (xy 173.99 104.14)
+		)
+		(stroke
+			(width 0)
+			(type solid)
+		)
+	)
+	(wire
+		(pts
+			(xy 59.69 82.55) (xy 59.69 78.74)
+		)
+		(stroke
+			(width 0)
+			(type solid)
+		)
+	)
+	(wire
+		(pts
+			(xy 229.87 96.52) (xy 237.49 96.52)
 		)
 		(stroke
@@
 	(polyline
 		(pts
-			(xy 18.415 63.246) (xy 277.114 63.246)
+			(xy 18.288 63.246) (xy 18.542 146.558)
 		)
 		(stroke
@@
 	(wire
 		(pts
-			(xy 80.01 78.74) (xy 80.01 82.55)
-		)
-		(stroke
-			(width 0)
-			(type default)
-		)
-	)
-	(wire
-		(pts
-			(xy 198.12 110.49) (xy 198.12 78.74)
-		)
-		(stroke
-			(width 0)
-			(type solid)
-		)
-	)
-	(wire
-		(pts
-			(xy 139.7 115.57) (xy 139.7 119.38)
-		)
-		(stroke
-			(width 0)
-			(type solid)
-		)
-	)
-	(wire
-		(pts
-			(xy 222.25 78.74) (xy 217.17 78.74)
-		)
-		(stroke
-			(width 0)
-			(type solid)
-		)
-	)
-	(wire
-		(pts
-			(xy 237.49 96.52) (xy 237.49 90.17)
-		)
-		(stroke
-			(width 0)
-			(type solid)
-		)
-	)
-	(wire
-		(pts
-			(xy 100.33 85.09) (xy 100.33 78.74)
-		)
-		(stroke
-			(width 0)
-			(type solid)
-		)
-	)
-	(wire
-		(pts
-			(xy 173.99 93.98) (xy 173.99 104.14)
-		)
-		(stroke
-			(width 0)
-			(type solid)
-		)
-	)
-	(wire
-		(pts
-			(xy 59.69 82.55) (xy 59.69 78.74)
-		)
-		(stroke
-			(width 0)
-			(type solid)
-		)
-	)
-	(wire
-		(pts
-			(xy 229.87 96.52) (xy 237.49 96.52)
-		)
-		(stroke
-			(width 0)
-			(type solid)
-		)
-	)
-	(polyline
-		(pts
-			(xy 18.288 63.246) (xy 18.542 146.558)
-		)
-		(stroke
-			(width 0)
-			(type dash)
-		)
-	)
-	(wire
-		(pts
-			(xy 237.49 78.74) (xy 247.65 78.74)
+			(xy 237.49 78.74) (xy 240.03 78.74)
 		)
 		(stroke
@@
 	(symbol
 		(lib_id "Connector:TestPoint")
-		(at 257.81 74.93 0)
+		(at 240.03 74.93 0)
 		(unit 1)
 		(exclude_from_sim no)
@@
 		(fields_autoplaced yes)
 		(property "Reference" "TP501"
-			(at 260.35 70.3579 0)
+			(at 242.57 70.3579 0)
 			(effects
 				(font
@@
 		)
 		(property "Value" "MPPT"
-			(at 260.35 72.8979 0)
+			(at 242.57 72.8979 0)
 			(effects
 				(font
@@
 		)
 		(property "Footprint" "TestPoint:TestPoint_Pad_D1.0mm"
-			(at 262.89 74.93 0)
+			(at 245.11 74.93 0)
 			(effects
 				(font
@@
 		)
 		(property "Datasheet" "~"
-			(at 262.89 74.93 0)
+			(at 245.11 74.93 0)
 			(effects
 				(font
@@
 		)
 		(property "Description" "test point"
-			(at 257.81 74.93 0)
+			(at 240.03 74.93 0)
 			(effects
 				(font
@@
 		)
 		(instances
-			(project ""
+			(project "govi_v3_SHT41_sensor_kicad"
 				(path "/ba95ddf4-72c6-4eeb-9c09-ae7c8e5af670/ae21eb8a-dcd5-4896-ab16-4532b352bb44"
 					(reference "TP501")

Commit message: "Routing done. DRC pending"
Parts:
- U501: footprint Package_SO:SSOP-10-1EP_3.9x4.9mm_P1mm_EP2.1x3.3mm_ThermalVias -> Package_SO:SSOP-10_3.9x4.9mm_P1.00mm
Changed lines of the file:
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@@
 			)
 		)
-		(property "Footprint" "Package_SO:SSOP-10-1EP_3.9x4.9mm_P1mm_EP2.1x3.3mm_ThermalVias"
+		(property "Footprint" "Package_SO:SSOP-10_3.9x4.9mm_P1.00mm"
 			(at 114.3 110.49 0)
 			(effects
